File: Ramsis.kicad_sch (KiCad schematic)
At the start: 0 parts

Commit message: update
Parts:
- added J1, J3, J4: Conn_01x03_Pin, Connector_PinHeader_1.00mm:PinHeader_1x03_P1.00mm_Vertical, symbol Connector:Conn_01x03_Pin
- added J2: Conn_01x04_Pin, Connector_PinHeader_1.00mm:PinHeader_1x04_P1.00mm_Vertical, symbol Connector:Conn_01x04_Pin
- added J5, J6: Conn_01x02_Pin, Connector_JST:JST_PH_S2B-PH-K_1x02_P2.00mm_Horizontal, symbol Connector:Conn_01x02_Pin
- added SW1: SW_Nidec_CAS-120A1, Button_Switch_THT:SW_Slide_SPDT_Angled_CK_OS102011MA1Q, symbol Switch:SW_Nidec_CAS-120A1
- added U1: ESP32-S3-DEVKITC-1-N8R2, Library:esp32 s55, symbol esp32 s355:ESP32-S3-DEVKITC-1-N8R2
- added U2: TP4056_MICRO-USB_CHARGER_-_1A, Library:MODULE_TP4056_MICRO-USB_CHARGER_-_1A, symbol charger55:TP4056_MICRO-USB_CHARGER_-_1A
- added U3: adafruit-MAX98357, max555:adafruit-MAX98357, symbol Max55555:adafruit-MAX98357
Connections:
- new net: J5.1 (Pin_1), U3.9 (OUTN)
- new net: J5.2 (Pin_2), U3.8 (OUTP)
- new net 3.3: J3.2 (Pin_2), U1.J1_1 (3V3), U1.J1_2 (3V3)
- new net BCLK: U1.J3_17 (GPIO47), U3.6 (BCLK)
- new net DIN: U1.J3_15 (GPIO45), U3.5 (DIN)
- new net GND: J1.3 (Pin_3), J2.4 (Pin_4), J3.3 (Pin_3), J4.1 (Pin_1), J6.1 (Pin_1), U1.J1_22 (GND), U1.J3_1 (GND), U1.J3_21 (GND), U1.J3_22 (GND), U2.BAT_N (BAT-), U2.OUT_N (OUT-), U3.2 (GND)
- new net LRC: U1.J3_16 (GPIO48), U3.7 (LRC)
- new net SCK: J1.1 (Pin_1), U1.J1_4 (GPIO4)
- new net SCL: J2.2 (Pin_2), U1.J1_15 (GPIO9)
- new net SD: J3.1 (Pin_1), U1.J1_6 (GPIO6)
- new net SDA: J2.1 (Pin_1), U1.J1_12 (GPIO8)
- new net SW1: J6.2 (Pin_2), SW1.1 (C)
- new net Touch: J4.3 (Pin_3), U1.J1_16 (GPIO10)
- new net VCC: J2.3 (Pin_3), SW1.3 (A), U1.J1_19 (GPIO13), U2.OUT_P (OUT+), U3.1 (Vin)
- new net Vcc: U2.BAT_P (BAT+)
- new net Ws: J1.2 (Pin_2), U1.J1_7 (GPIO7)
Other:
- note added: "Battery"
- note added: "Companion in daily life_showing time and weather"
- note added: "Description"
- note added: "ESP"
- note added: "ESP Connection"
- note added: "INMP441"
- note added: "MAX98357 I2S"
- note added: "Microphone"
- note added: "OLED"
- note added: "Power"
- note added: "Ramasis Robot"
- note added: "Sound"
- note added: "Speakers"
- note added: "TP4056"
- note added: "TTP223-B"
- note added: "Touch Sensor"
- note added: "oled 1.3"

Commit message: update
Parts:
- added H1: MountingHole, MountingHole:MountingHole_3.2mm_M3, symbol Mechanical:MountingHole
Changed lines of the file:
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@@
+	)
+	(symbol
+		(lib_id "Mechanical:MountingHole")
+		(at 242.57 106.68 0)
+		(unit 1)
+		(exclude_from_sim no)
+		(in_bom no)
+		(on_board yes)
+		(dnp no)
+		(fields_autoplaced yes)
+		(property "Reference" "H1"
+			(at 245.11 105.4099 0)
+			(effects
+				(font
+					(size 1.27 1.27)
+				)
+				(justify left)
+			)
+		)
+		(property "Value" "MountingHole"
+			(at 245.11 107.9499 0)
+			(effects
+				(font
+					(size 1.27 1.27)
+				)
+				(justify left)
+			)
+		)
+		(property "Footprint" "MountingHole:MountingHole_3.2mm_M3"
+			(at 242.57 106.68 0)
+			(effects
+				(font
+					(size 1.27 1.27)
+				)
+				(hide yes)
+			)
+		)
+		(property "Datasheet" "~"
+			(at 242.57 106.68 0)
+			(effects
+				(font
+					(size 1.27 1.27)
+				)
+				(hide yes)
+			)
+		)
+		(property "Description" "Mounting Hole without connection"
+			(at 242.57 106.68 0)
+			(effects
+				(font
+					(size 1.27 1.27)
+				)
+				(hide yes)
+			)
+		)
+		(instances
+			(project ""
+				(path "/358999d6-3183-4327-aa1f-0022f87f5165"
+					(reference "H1")
+					(unit 1)
+				)
+			)
+		)
 	)
 	(symbol
