File: Ramsis/Ramsis.kicad_pcb (KiCad board)
At the start: 2 copper layers, 113.5 x 86.5 mm, 14 parts, among them J1 Conn_01x03_Pin, J2 Conn_01x04_Pin, J3 Conn_01x03_Pin, J4 Conn_01x03_Pin, J5 Conn_01x02_Pin, J6 Conn_01x02_Pin, SW1 SW_Nidec_CAS-120A1, U1 ESP32-S3-DEVKITC-1-N8R2, U2 TP4056_MICRO-USB_CHARGER_-_1A, U3 adafruit-MAX98357

Commit message: update
Parts:
- J1, J3, J4: footprint Connector_PinHeader_1.00mm:PinHeader_1x03_P1.00mm_Vertical -> Connector_PinHeader_2.00mm:PinHeader_1x03_P2.00mm_Vertical
- J2: footprint Connector_PinHeader_1.00mm:PinHeader_1x04_P1.00mm_Vertical -> Connector_PinHeader_2.00mm:PinHeader_1x04_P2.00mm_Vertical
- J6: moved to F.Cu
- turned J6 to 180 degrees
Routing:
- net SW1: track 51.5 -> 56.4 mm
- net GND: track 110.2 -> 106.5 mm
- net VCC: track 212.8 -> 214.9 mm
- net SCL: track 71.6 -> 69.7 mm, vias 0 -> 1
- net SD: track 35.0 -> 36.9 mm
- net 3.3: track 27.3 -> 26.3 mm
- net Touch: track 63.2 -> 64.0 mm
